Commit message: Stripped down imprimis sim, renamed dynamic transform example to orbit pkg and parameterized it

File: src/imprimis_sim_description/urdf/diffbot.ros2_control.xacro (robot description, xacro)
@@ -1,20 +1,12 @@
 <?xml version="1.0"?>
 <robot xmlns:xacro="http://www.ros.org/wiki/xacro">
-  <xacro:macro name="diffbot_ros2_control" params="name hardware_type">
+  <xacro:macro name="diffbot_ros2_control" params="name">
     <ros2_control name="${name}" type="system">
-      <!-- Fake hardware-->
-      <xacro:if value="${hardware_type == 'fake'}">
-        <hardware>
-          <plugin>mock_components/GenericSystem</plugin>
-          <param name="calculate_dynamics">true</param>
-        </hardware>
-      </xacro:if>
-      <!-- Gazebo-simulated Hardware -->
-      <xacro:if value="${hardware_type == 'simulated'}">
-        <hardware>
-          <plugin>gz_ros2_control/GazeboSimSystem</plugin>
-        </hardware>
-      </xacro:if>
-      <!-- Joint definitions -->
+      <!-- Fake hardware plugin-->
+      <hardware>
+        <plugin>mock_components/GenericSystem</plugin>
+        <param name="calculate_dynamics">true</param>
+      </hardware>
+      <!-- Define which joints in the urdf can move -->
       <joint name="left_wheel_joint">
         <command_interface name="velocity"/>
@@ -27,16 +19,4 @@
         <state_interface name="velocity"/>
       </joint>
-      <!-- Arbitrary state interfaces (GPIOs)-->
-      <gpio name="imprimis_data">
-        <command_interface name="dummy_gpio_cmd"/>
-        <state_interface name="imuHeading"/>
-        <state_interface name="manualMode"/>
-        <state_interface name="boardBConnected"/>
-        <state_interface name="gpsFix"/>
-        <state_interface name="gpsLat"/>
-        <state_interface name="gpsLong"/>
-        <state_interface name="gpsAlt"/>
-        <state_interface name="gpsHdop"/>
-      </gpio>
     </ros2_control>
   </xacro:macro>

File: src/imprimis_sim_description/urdf/diffbot.urdf.xacro (robot description, xacro)
@@ -1,7 +1,4 @@
 <?xml version="1.0"?>
-<!-- Basic differential drive mobile base -->
 <robot xmlns:xacro="http://www.ros.org/wiki/xacro" name="diffdrive_robot">
-  <xacro:arg name="hardware_type" default="simulated" />
-  <xacro:arg name="publish_odom_tf" default="true" />
   <!-- Import and expand core robot description -->
   <xacro:include filename="$(find imprimis_sim_description)/urdf/diffbot_description.urdf.xacro" />
@@ -11,7 +8,4 @@
   <!-- Import and expand diffbot ros2_control description -->
   <xacro:include filename="$(find imprimis_sim_description)/urdf/diffbot.ros2_control.xacro" />
-  <xacro:diffbot_ros2_control name="DiffBot" hardware_type="$(arg hardware_type)"/>
-  <!-- Import and expand gazebo information. It's fine to keep it in there even if hardware type isn't simulated. -->
-  <xacro:include filename="$(find imprimis_sim_description)/urdf/gazebo_info.xacro"/>
-  <xacro:gzinfo publish_odom_tf="$(arg publish_odom_tf)"/>
+  <xacro:diffbot_ros2_control name="DiffBot"/>
 </robot>
